File: PCB/Gantry_PCBv2/Gantry_PCBv2.kicad_pcb (KiCad board)
At the start: 2 copper layers, 120 x 120 mm, 64 parts, among them J1 Conn_01x14, J10 B2B-XH-A_LF__SN_, J11 B2B-XH-A_LF__SN_, J12 B2B-XH-A_LF__SN_, J13 Conn_01x03_Pin, J17 B2B-XH-A_LF__SN_, J2 Conn_01x14, J20 TYPE-C-31-M-12, J3 Conn_01x10, J4 Screw_Terminal_01x02, J5 DCJ200-10-A-XX-X_REVA, J6 Conn_01x04_Pin, J7 Conn_01x04_Pin, J8 Conn_01x04_Pin, J9 Conn_01x04_Pin, Q1 SS8050, Q2 SS8050, SW7 SW_0, SW8 SW_EN, U1 ESP32-WROOM-32E, U2 CH340C, U3 TB6612FNG H-bridge Motor Driv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, U4 LM2576S-5, U5 AMS1117-3.3, U6 DRV8825_STEPPER_MOTOR_DRIVER_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, U7 DRV8825_STEPPER_MOTOR_DRIVER_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, U8 DRV8825_STEPPER_MOTOR_DRIVER_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, U9 DRV8825_STEPPER_MOTOR_DRIVER_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

Commit message: PCB continued
Connections:
- J3 pad 3: /SD2 -> unconnected-(J3-Pin_3-Pad3)
- J3 pad 4: /SD3 -> unconnected-(J3-Pin_4-Pad4)
- J3 pad 5: /CMD -> unconnected-(J3-Pin_5-Pad5)
- J3 pad 6: /CLK -> unconnected-(J3-Pin_6-Pad6)
- J3 pad 7: /SD0 -> unconnected-(J3-Pin_7-Pad7)
- J3 pad 8: /SD1 -> unconnected-(J3-Pin_8-Pad8)
Changed lines of the file:
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@@
 	(net 34 "/RXD")
 	(net 35 "/5")
-	(net 36 "/SD1")
-	(net 37 "/CMD")
-	(net 38 "/SD2")
+	(net 36 "unconnected-(J3-Pin_6-Pad6)")
+	(net 37 "unconnected-(J3-Pin_8-Pad8)")
+	(net 38 "unconnected-(J3-Pin_3-Pad3)")
 	(net 39 "/2")
-	(net 40 "/SD3")
-	(net 41 "/SD0")
+	(net 40 "unconnected-(J3-Pin_4-Pad4)")
+	(net 41 "unconnected-(J3-Pin_7-Pad7)")
 	(net 42 "/15")
-	(net 43 "/CLK")
+	(net 43 "unconnected-(J3-Pin_5-Pad5)")
 	(net 44 "/13")
 	(net 45 "/SM2_A1")
@@
 			(net 91 "unconnected-(U7-~{FLT}-Pad10)")
 			(pinfunction "~{FLT}")
-			(pintype "output")
+			(pintype "output+no_connect")
 			(solder_mask_margin 0.102)
 		)
@@
 			(layers "*.Cu" "*.Mask")
 			(remove_unused_layers no)
-			(net 38 "/SD2")
+			(net 38 "unconnected-(J3-Pin_3-Pad3)")
 			(pinfunction "Pin_3")
-			(pintype "passive")
+			(pintype "passive+no_connect")
 		)
 		(pad "4" thru_hole circle
@@
 			(layers "*.Cu" "*.Mask")
 			(remove_unused_layers no)
-			(net 40 "/SD3")
+			(net 40 "unconnected-(J3-Pin_4-Pad4)")
 			(pinfunction "Pin_4")
-			(pintype "passive")
+			(pintype "passive+no_connect")
 		)
 		(pad "5" thru_hole circle
@@
 			(layers "*.Cu" "*.Mask")
 			(remove_unused_layers no)
-			(net 37 "/CMD")
+			(net 43 "unconnected-(J3-Pin_5-Pad5)")
 			(pinfunction "Pin_5")
-			(pintype "passive")
+			(pintype "passive+no_connect")
 		)
 		(pad "6" thru_hole circle
@@
 			(layers "*.Cu" "*.Mask")
 			(remove_unused_layers no)
-			(net 43 "/CLK")
+			(net 36 "unconnected-(J3-Pin_6-Pad6)")
 			(pinfunction "Pin_6")
-			(pintype "passive")
+			(pintype "passive+no_connect")
 		)
 		(pad "7" thru_hole circle
@@
 			(layers "*.Cu" "*.Mask")
 			(remove_unused_layers no)
-			(net 41 "/SD0")
+			(net 41 "unconnected-(J3-Pin_7-Pad7)")
 			(pinfunction "Pin_7")
-			(pintype "passive")
+			(pintype "passive+no_connect")
 		)
 		(pad "8" thru_hole circle
@@
 			(layers "*.Cu" "*.Mask")
 			(remove_unused_layers no)
-			(net 36 "/SD1")
+			(net 37 "unconnected-(J3-Pin_8-Pad8)")
 			(pinfunction "Pin_8")
-			(pintype "passive")
+			(pintype "passive+no_connect")
 		)
 		(pad "9" thru_hole circle
@@
 			(net 93 "unconnected-(U9-~{FLT}-Pad10)")
 			(pinfunction "~{FLT}")
-			(pintype "output")
+			(pintype "output+no_connect")
 			(solder_mask_margin 0.102)
 		)
@@
 			(net 90 "unconnected-(U6-~{FLT}-Pad10)")
 			(pinfunction "~{FLT}")
-			(pintype "output")
+			(pintype "output+no_connect")
 			(solder_mask_margin 0.102)
 		)
@@
 			(net 61 "unconnected-(J13-Pin_1-Pad1)")
 			(pinfunction "Pin_1")
-			(pintype "passive")
+			(pintype "passive+no_connect")
 		)
 		(pad "2" thru_hole oval
@@
 			(net 92 "unconnected-(U8-~{FLT}-Pad10)")
 			(pinfunction "~{FLT}")
-			(pintype "output")
+			(pintype "output+no_connect")
 			(solder_mask_margin 0.102)
 		)

Commit message: Changed Footprints
Parts:
- removed J20: TYPE-C-31-M-12, Connector_USB:USB_C_Receptacle_HRO_TYPE-C-31-M-12
- removed R6, R7: 5.1K, Resistor_SMD:R_0805_2012Metric
- added J14: USB_C_Receptacle_USB2.0_16P, Connector_USB:USB_C_Receptacle_HRO_TYPE-C-31-M-12, F.Cu at (151.9, 53.3)
- added R10: 5.1K, Resistor_SMD:R_0805_2012Metric, F.Cu at (143.2, 63.2)
- added R11: 5.1K, Resistor_SMD:R_0805_2012Metric, F.Cu at (143.2, 58.2)
- U3: footprint motor_driver:TB6612FNG -> Motor Drivers:MODULE_ROB-14450
