File: PCB/Gantry_PCBv2/Gantry_PCBv2.kicad_pcb (KiCad board)
At the start: 2 copper layers, 120 x 120 mm, 64 parts, among them J1 Conn_01x14, J10 B2B-XH-A_LF__SN_, J11 B2B-XH-A_LF__SN_, J12 B2B-XH-A_LF__SN_, J13 Conn_01x03_Pin, J14 USB_C_Receptacle_USB2.0_16P, J17 B2B-XH-A_LF__SN_, J2 Conn_01x14, J3 Conn_01x10, J4 Screw_Terminal_01x02, J5 DCJ200-10-A-XX-X_REVA, J6 Conn_01x04_Pin, J7 Conn_01x04_Pin, J8 Conn_01x04_Pin, J9 Conn_01x04_Pin, Q1 SS8050, Q2 SS8050, SW7 SW_0, SW8 SW_EN, U1 ESP32-WROOM-32E, U2 CH340C, U3 TB6612FNG H-bridge Motor Driv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, U4 LM2576S-5, U5 AMS1117-3.3, U6 DRV8825_STEPPER_MOTOR_DRIVER_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, U7 DRV8825_STEPPER_MOTOR_DRIVER_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, U8 DRV8825_STEPPER_MOTOR_DRIVER_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, U9 DRV8825_STEPPER_MOTOR_DRIVER_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

Commit message: Added MCP23017 GPIO Expander and Joystick
Parts:
- removed the C14 at (138.0, 136.0)
- removed the C7 at (65.5, 91.0)
- removed the J13 at (165.0, 111.0)
- removed the J14 at (151.9, 53.3)
- removed the U5 at (91.0, 79.2)
- added C15: 1uF, Capacitor_SMD:C_0805_2012Metric, F.Cu at (265.0, 88.5)
- added C16: 4.7uF, Capacitor_SMD:C_0805_2012Metric, F.Cu at (265.0, 91.5)
- added C18: 100n, Capacitor_SMD:CP_Elec_6.3x7.7, F.Cu at (222.0, 57.6)
- added C19: 100n, Capacitor_SMD:CP_Elec_6.3x7.7, F.Cu at (222.0, 65.8)
- added C2: 10uF, Capacitor_SMD:C_0805_2012Metric, F.Cu at (260.5, 79.5)
- added C21: 470u, Capacitor_SMD:CP_Elec_6.3x7.7, F.Cu at (222.0, 73.9)
- added C22: 100n, Capacitor_SMD:CP_Elec_6.3x7.7, F.Cu at (232.4, 57.6)
- added C23: 100n, Capacitor_SMD:CP_Elec_6.3x7.7, F.Cu at (232.4, 65.8)
- added C24: 100n, Capacitor_SMD:CP_Elec_6.3x7.7, F.Cu at (232.4, 73.9)
- added C25: 470u, Capacitor_SMD:CP_Elec_6.3x7.7, F.Cu at (242.9, 57.6)
- added C26: 470u, Capacitor_SMD:CP_Elec_6.3x7.7, F.Cu at (242.9, 65.8)
- added C27: 100n, Capacitor_SMD:CP_Elec_6.3x7.7, F.Cu at (242.9, 73.9)
- added C28: 100n, Capacitor_SMD:CP_Elec_6.3x7.7, F.Cu at (4.69, 30.6)
- added C3: 150pF, Capacitor_SMD:C_0805_2012Metric, F.Cu at (260.5, 82.5)
- added C4: 100nF, Capacitor_SMD:C_0805_2012Metric, F.Cu at (260.5, 85.5)
- added D1: SS34, Diode_SMD:D_SMB, F.Cu at (252.3, 71.1)
- added D10: B_LED, LED_SMD:LED_0201_0603Metric_Pad0.64x0.40mm_HandSolder, F.Cu at (256.9, 84.1)
- added D11: Y_LED, LED_SMD:LED_0201_0603Metric_Pad0.64x0.40mm_HandSolder, F.Cu at (256.9, 85.9)
- added D12: SS14, Diode_SMD:D_SMA, F.Cu at (261.0, 73.1)
- added D16: Y_LED, LED_SMD:LED_0201_0603Metric_Pad0.64x0.40mm_HandSolder, F.Cu at (256.9, 92.9)
- added D17: Y_LED, LED_SMD:LED_0201_0603Metric_Pad0.64x0.40mm_HandSolder, F.Cu at (256.9, 94.6)
- added D2: SS14, Diode_SMD:D_SMA, F.Cu at (261.0, 68.5)
- added D3: LED, LED_SMD:LED_0603_1608Metric_Pad1.05x0.95mm_HandSolder, F.Cu at (265.0, 94.3)
- added D4: D_Schottky, Diode_SMD:D_SMA_Handsoldering, F.Cu at (262.0, 55.8)
- added D5: LED, LED_SMD:LED_0603_1608Metric_Pad1.05x0.95mm_HandSolder, F.Cu at (265.0, 96.9)
- added D6: R_LED, LED_SMD:LED_0201_0603Metric_Pad0.64x0.40mm_HandSolder, F.Cu at (256.9, 78.9)
- added D7: G_LED, LED_SMD:LED_0201_0603Metric_Pad0.64x0.40mm_HandSolder, F.Cu at (256.9, 80.6)
- added D8: B_LED, LED_SMD:LED_0201_0603Metric_Pad0.64x0.40mm_HandSolder, F.Cu at (256.9, 82.4)
- added D9: SP0503BAHT, Package_TO_SOT_SMD:SOT-143, F.Cu at (230.6, 100.3)
- added F1: 3A, Fuse:Fuse_Littelfuse-LVR100, F.Cu at (221.2, 81.3)
- added F2: 1A, Fuse:Fuse_Littelfuse-LVR100, F.Cu at (221.2, 88.0)
- added F3: Polyfuse, Fuse:Fuse_Littelfuse-LVR100, F.Cu at (3.89, 16.6)
- added J11: USB_C_Receptacle_USB2.0_16P, Connector_USB:USB_C_Receptacle_GCT_USB4105-xx-A_16P_TopMnt_Horizontal, F.Cu at (222.6, 96.6)
- added J16: Conn_01x05_Pin, Connector_PinHeader_2.54mm:PinHeader_1x05_P2.54mm_Vertical, F.Cu at (27.4, -1.40)
- added J17: Conn_01x05_Pin, Connector_PinHeader_2.54mm:PinHeader_1x05_P2.54mm_Vertical, F.Cu at (32.0, -1.40)
- added J3: Conn_01x03_Pin, Connector_JST:JST_EH_B3B-EH-A_1x03_P2.50mm_Vertical, F.Cu at (244.5, 98.3)
- added Q1: NMOS, Package_TO_SOT_THT:TO-247-3_Vertical, F.Cu at (2.74, 23.0)
- added R12: 40.2k, Resistor_SMD:R_0805_2012Metric_Pad1.20x1.40mm_HandSolder, F.Cu at (248.1, 79.5)
- added R13: 1K, Resistor_SMD:R_0805_2012Metric_Pad1.20x1.40mm_HandSolder, F.Cu at (248.1, 82.4)
- added R14: 1K, Resistor_SMD:R_0805_2012Metric_Pad1.20x1.40mm_HandSolder, F.Cu at (248.1, 85.4)
- added R15: 1K, Resistor_SMD:R_0805_2012Metric_Pad1.20x1.40mm_HandSolder, F.Cu at (248.1, 88.3)
- added R16: 10K, Resistor_SMD:R_0805_2012Metric_Pad1.20x1.40mm_HandSolder, F.Cu at (248.1, 91.3)
- added R17: 10K, Resistor_SMD:R_0805_2012Metric_Pad1.20x1.40mm_HandSolder, F.Cu at (248.1, 94.2)
- added R18: 10K, Resistor_SMD:R_0805_2012Metric_Pad1.20x1.40mm_HandSolder, F.Cu at (252.9, 79.5)
- added R2: 100k, Resistor_SMD:R_0805_2012Metric_Pad1.20x1.40mm_HandSolder, F.Cu at (243.4, 79.5)
- added R21: 4.7k, Resistor_SMD:R_0805_2012Metric, F.Cu at (250.3, 55.0)
- added R22: 1.5k, Resistor_SMD:R_0805_2012Metric, F.Cu at (250.3, 58.0)
- added R23: 100, Resistor_SMD:R_0603_1608Metric, F.Cu at (239.0, 79.2)
- added R24: 100, Resistor_SMD:R_0603_1608Metric, F.Cu at (239.0, 81.8)
- added R25: 100, Resistor_SMD:R_0603_1608Metric, F.Cu at (239.0, 84.3)
- added R26: 100, Resistor_SMD:R_0603_1608Metric, F.Cu at (239.0, 86.8)
- added R27: 150, Resistor_SMD:R_0805_2012Metric, F.Cu at (250.3, 60.9)
- added R28: 5.1K, Resistor_SMD:R_0805_2012Metric_Pad1.20x1.40mm_HandSolder, F.Cu at (252.9, 82.4)
- added R29: 5.1K, Resistor_SMD:R_0805_2012Metric_Pad1.20x1.40mm_HandSolder, F.Cu at (252.9, 85.4)
- added R3: 24.9k, Resistor_SMD:R_0805_2012Metric_Pad1.20x1.40mm_HandSolder, F.Cu at (243.4, 82.4)
- added R30: 150, Resistor_SMD:R_0805_2012Metric, F.Cu at (250.3, 63.9)
- added R31: 600, Resistor_SMD:R_0805_2012Metric, F.Cu at (250.3, 66.8)
- added R32: 600, Resistor_SMD:R_0805_2012Metric, F.Cu at (254.7, 55.0)
- added R35: 600, Resistor_SMD:R_0805_2012Metric, F.Cu at (254.7, 58.0)
- added R36: 100, Resistor_SMD:R_0603_1608Metric, F.Cu at (239.0, 89.3)
- added R37: 100, Resistor_SMD:R_0603_1608Metric, F.Cu at (239.0, 91.8)
- added R38: 100, Resistor_SMD:R_0603_1608Metric, F.Cu at (239.0, 94.3)
- added R39: 100, Resistor_SMD:R_0603_1608Metric, F.Cu at (239.0, 96.8)
- added R4: 100k, Resistor_SMD:R_0805_2012Metric_Pad1.20x1.40mm_HandSolder, F.Cu at (243.4, 85.4)
- added R40: 600, Resistor_SMD:R_0805_2012Metric, F.Cu at (254.7, 60.9)
- added R41: 600, Resistor_SMD:R_0805_2012Metric, F.Cu at (254.7, 63.9)
- added R42: 600, Resistor_SMD:R_0805_2012Metric, F.Cu at (254.7, 66.8)
- added R43: 100k, Resistor_SMD:R_0805_2012Metric_Pad1.20x1.40mm_HandSolder, F.Cu at (35.0, 14.8)
- added R44: 100k, Resistor_SMD:R_0805_2012Metric_Pad1.20x1.40mm_HandSolder, F.Cu at (35.0, 17.7)
- added R45: 100k, Resistor_SMD:R_0805_2012Metric_Pad1.20x1.40mm_HandSolder, F.Cu at (35.0, 20.6)
- added R46: 100k, Resistor_SMD:R_0805_2012Metric_Pad1.20x1.40mm_HandSolder, F.Cu at (35.0, 23.6)
- added R47: 100k, Resistor_SMD:R_0805_2012Metric_Pad1.20x1.40mm_HandSolder, F.Cu at (35.0, 26.6)
- added R48: 100k, Resistor_SMD:R_0805_2012Metric_Pad1.20x1.40mm_HandSolder, F.Cu at (35.0, 29.5)
- added R5: 100k, Resistor_SMD:R_0805_2012Metric_Pad1.20x1.40mm_HandSolder, F.Cu at (243.4, 88.3)
- added R6: 10k, Resistor_SMD:R_0815_2038Metric, F.Cu at (260.5, 95.8)
- added R7: 1.2k, Resistor_SMD:R_0805_2012Metric_Pad1.20x1.40mm_HandSolder, F.Cu at (243.4, 91.3)
- added TH1: 10k, Resistor_SMD:R_0805_2012Metric_Pad1.20x1.40mm_HandSolder, F.Cu at (252.9, 88.3)
- added TP1: TP, TestPoint:TestPoint_Pad_D2.0mm, F.Cu at (155.0, 118.0)
- added TP2: TP, TestPoint:TestPoint_Pad_D2.0mm, F.Cu at (155.0, 121.3)
- added TP3: TP, TestPoint:TestPoint_Pad_D2.0mm, F.Cu at (155.0, 124.7)
- added TP4: TP, TestPoint:TestPoint_Pad_D2.0mm, F.Cu at (155.0, 128.1)
- added TP5: TP, TestPoint:TestPoint_Pad_D2.0mm, F.Cu at (155.0, 131.4)
- added TP6: TP, TestPoint:TestPoint_Pad_D2.0mm, F.Cu at (155.0, 134.8)
- added TP7: TP, TestPoint:TestPoint_Pad_D2.0mm, F.Cu at (155.0, 138.1)
- added TP8: TP, TestPoint:TestPoint_Pad_D2.0mm, F.Cu at (155.0, 141.4)
- added U10: 74HC245, Package_SO:SOIC-20W_7.5x15.4mm_P1.27mm, F.Cu at (5.87, 4.79)
- added U11: 74HC245, Package_SO:SOIC-20W_7.5x15.4mm_P1.27mm, F.Cu at (18.7, 4.79)
- added U12: MCP23017_SO, Package_SO:SOIC-28W_7.5x17.9mm_P1.27mm, F.Cu at (26.2, 23.1)
- added U2: MP1584, Package_SO:SOIC-8-1EP_3.9x4.9mm_P1.27mm_EP2.41x3.3mm, F.Cu at (232.7, 94.7)
- C10: value 0.1uF -> 100nF
- C11: value 22uF -> 100nF; footprint Capacitor_SMD:C_0805_2012Metric -> Capacitor_SMD:C_01005_0402Metric
- C12: value 100u -> 100nF; footprint Capacitor_SMD:CP_Elec_6.3x7.7 -> Capacitor_SMD:C_01005_0402Metric
- C13: value 100u -> 0.1uF; footprint Capacitor_SMD:CP_Elec_6.3x7.7 -> Capacitor_SMD:C_0805_2012Metric
- C20: renamed from C15; value 100u -> 470u
- C6: value 100uF -> NS; footprint Capacitor_SMD:CP_Elec_6.3x7.7 -> Capacitor_SMD:C_0805_2012Metric
- C8: value 10uF -> 22uF
- C9: value 0.1uF -> 1uF
- D13: value SS14 -> Y_LED; footprint Diode_SMD:D_SMA -> LED_SMD:LED_0201_0603Metric_Pad0.64x0.40mm_HandSolder
- D14: value SS24 -> Y_LED; footprint Diode_SMD:D_SMA -> LED_SMD:LED_0201_0603Metric_Pad0.64x0.40mm_HandSolder
- D15: value SS34 -> Y_LED; footprint Diode_SMD:D_SMB -> LED_SMD:LED_0201_0603Metric_Pad0.64x0.40mm_HandSolder
- L1: value 100uH -> 15uH; footprint Inductor_SMD:L_10.4x10.4_H4.8 -> Inductor_SMD:L_Sunlord_MWSA0603S
- R10: value 5.1K -> 330; footprint Resistor_SMD:R_0805_2012Metric -> Resistor_SMD:R_0603_1608Metric_Pad0.98x0.95mm_HandSolder
- R11: value 5.1K -> 210k; footprint Resistor_SMD:R_0805_2012Metric -> Resistor_SMD:R_0805_2012Metric_Pad1.20x1.40mm_HandSolder
- U1: footprint ESP32-WROOM:XCVR_ESP32-WROOM-32E__4MB_HIGH_TEMP_ -> RF_Module:ESP32-WROOM-32E
- U4: value LM2576S-5 -> TLV75733PDBV; footprint Package_TO_SOT_SMD:TO-263-5_TabPin3 -> Package_TO_SOT_SMD:SOT-23-5
- U5: renamed from U8; footprint DRV8825_STEPPER_MOTOR_DRIVER_CARRIER (1):IC_DRV8825_STEPPER_MOTOR_DRIVER_CARRIER -> StepperMotor Driver:stepper
- U6: renamed from U9; footprint DRV8825_STEPPER_MOTOR_DRIVER_CARRIER (1):IC_DRV8825_STEPPER_MOTOR_DRIVER_CARRIER -> StepperMotor Driver:stepper
- U8: renamed from U6; footprint DRV8825_STEPPER_MOTOR_DRIVER_CARRIER (1):IC_DRV8825_STEPPER_MOTOR_DRIVER_CARRIER -> StepperMotor Driver:stepper
- U9: renamed from U7; footprint DRV8825_STEPPER_MOTOR_DRIVER_CARRIER (1):IC_DRV8825_STEPPER_MOTOR_DRIVER_CARRIER -> StepperMotor Driver:stepper
- moved C6 203.8 mm to (260.5, 88.5), turned to 0 degrees
- moved D14 201.3 mm to (256.9, 89.4), turned to 0 degrees
- moved L1 192.5 mm to (261.9, 62.2), turned to 0 degrees
- moved U4 188.6 mm to (260.9, 101.0), turned to 0 degrees
- moved D15 179.4 mm to (256.9, 91.1), turned to 0 degrees
- moved C10 174.3 mm to (265.0, 82.5), turned to 0 degrees
- moved C9 173.7 mm to (265.0, 79.5), turned to 0 degrees
- moved C8 169.0 mm to (260.5, 91.5), turned to 0 degrees
- moved C11 162.8 mm to (253.6, 74.7), turned to 0 degrees
- moved C13 157.8 mm to (265.0, 85.5), turned to 0 degrees
- moved C12 118.4 mm to (253.6, 76.3), turned to 0 degrees
- moved R10 102.0 mm to (250.3, 75.1)
- moved D13 97.5 mm to (256.9, 87.6), turned to 0 degrees
- moved R11 93.6 mm to (243.4, 94.2)
- renumbered C4 to C14, C5 to C17, C2 to C5, C3 to C7, H5 to H1, H6 to H2, H7 to H3, H8 to H4, H1 to H5, H2 to H6, H3 to H7, H4 to H8, J4 to J1, J17 to J10, J6 to J12, J7 to J13, J8 to J14, J9 to J15, J5 to J2, J1 to J4, J10 to J5, J11 to J6, J12 to J7, J2 to J8, J3 to J9, Q1 to Q2, Q2 to Q3, R4 to R19, R5 to R20, R8 to R33, R9 to R34, R2 to R8, R3 to R9, SW7 to SW1, SW8 to SW2, U2 to U3, U3 to U7
Connections:
- C10 pad 1: /3V3 -> Net-(C10-Pad1)
- C11 pad 1: /3V3 -> Net-(C11-Pad1)
- C12 pad 1: /12V_P -> Net-(C12-Pad1)
- C13 pad 1: /12V_P -> /5V_R
- C20 pad 1: /12V_P -> /12V_R
- C6 pad 1: Net-(D14-K) -> Net-(U2-COMP)
- C9 pad 1: /5V -> /5V_R
- D13 pad 1: /5V -> GND
- D13 pad 2: /VBUSC -> Net-(D13-A)
- D14 pad 1: Net-(D14-K) -> GND
- D14 pad 2: /12V -> Net-(D14-A)
- D15 pad 1: Net-(D15-K) -> GND
- D15 pad 2: GND -> Net-(D15-A)
- J5 pad 1: /15 -> Net-(C12-Pad1)
- J6 pad 1: /19 -> Net-(C10-Pad1)
- J7 pad 1: /18 -> Net-(C11-Pad1)
- L1 pad 1: Net-(D15-K) -> Net-(D4-K)
- R10 pad 2: /CC2 -> Net-(D5-K)
- R11 pad 1: /CC1 -> /5V
- R11 pad 2: GND -> /FB
- R33 pad 1: /34 -> /18
- R34 pad 1: /35 -> /19
- U4 pad 1: Net-(D14-K) -> /5V_R
- U4 pad 2: Net-(D15-K) -> GND
- U4 pad 3: GND -> /5V_R
- U4 pad 4: /5V -> unconnected-(U4-NC-Pad4)
- U4 pad 5: GND -> /3V3
- U5 pad 16: /12V_P -> /12V_R
- U5 pad 7: /26 -> Net-(U5-STEP)
- U5 pad 8: /25 -> Net-(U5-DIR)
- U6 pad 16: /12V_P -> /12V_R
- U6 pad 7: /12 -> Net-(U6-STEP)
- U6 pad 8: /14 -> Net-(U6-DIR)
- U8 pad 16: /12V_P -> /12V_R
- U8 pad 7: /23 -> Net-(U8-STEP)
- U8 pad 8: /22 -> Net-(U8-DIR)
- U9 pad 16: /12V_P -> /12V_R
- U9 pad 7: /26 -> Net-(U9-STEP)
- U9 pad 8: /25 -> Net-(U9-DIR)
Routing:
- net (no net): track 0.00 -> 134.1 mm
- net Net-(D14-K): track 75.9 -> 0.00 mm
- net Net-(D15-K): track 29.1 -> 0.00 mm
- net /VBUSC: track 16.8 -> 0.00 mm
- net /CC1: track 6.53 -> 0.00 mm
- net /CC2: track 5.77 -> 0.00 mm

Commit message: Minor Changes in Schematic, Initial Layout of PCB done
Parts:
- removed C1, C5, C7: 0.1uF, Capacitor_SMD:C_0805_2012Metric
- removed D3, D5: LED, LED_SMD:LED_0603_1608Metric_Pad1.05x0.95mm_HandSolder
- removed R10: 330, Resistor_SMD:R_0603_1608Metric_Pad0.98x0.95mm_HandSolder
- removed R7: 1.2k, Resistor_SMD:R_0805_2012Metric_Pad1.20x1.40mm_HandSolder
- removed U1: ESP32-WROOM-32E, RF_Module:ESP32-WROOM-32E
- removed U3: CH340C, Package_SO:SOIC-16_3.9x9.9mm_P1.27mm
- added C29: 10uF, Capacitor_SMD:C_0805_2012Metric_Pad1.18x1.45mm_HandSolder, F.Cu at (107.8, 91.0)
- added C30: 0.1uF, Capacitor_SMD:C_0805_2012Metric_Pad1.18x1.45mm_HandSolder, F.Cu at (110.0, 88.5)
- added C31: 4.7u, Capacitor_SMD:C_0805_2012Metric_Pad1.18x1.45mm_HandSolder, F.Cu at (71.0, 39.8)
- added C32: 0.1u, Capacitor_SMD:C_0805_2012Metric_Pad1.18x1.45mm_HandSolder, F.Cu at (71.0, 43.8)
- added C33: 0.1uF, Capacitor_SMD:C_0805_2012Metric_Pad1.18x1.45mm_HandSolder, F.Cu at (59.5, 101.0)
- added D18: LED, LED_SMD:LED_0805_2012Metric_Pad1.15x1.40mm_HandSolder, F.Cu at (92.2, 27.0)
- added D19: LED, LED_SMD:LED_0805_2012Metric_Pad1.15x1.40mm_HandSolder, F.Cu at (92.2, 29.5)
- added JP1: SolderJumper, Jumper:SolderJumper-3_P1.3mm_Open_Pad1.0x1.5mm_NumberLabels, F.Cu at (128.1, 97.5)
- added JP2: SolderJumper, Jumper:SolderJumper-3_P1.3mm_Open_Pad1.0x1.5mm_NumberLabels, F.Cu at (128.0, 92.0)
- added JP3: SolderJumper, Jumper:SolderJumper-3_P1.3mm_Open_Pad1.0x1.5mm_NumberLabels, F.Cu at (127.8, 86.0)
- added R49: 1K, Resistor_SMD:R_0805_2012Metric_Pad1.20x1.40mm_HandSolder, F.Cu at (82.5, 69.2)
- added R50: 10k, Resistor_SMD:R_0805_2012Metric_Pad1.20x1.40mm_HandSolder, F.Cu at (112.5, 103.5)
- added R51: 10k, Resistor_SMD:R_0805_2012Metric_Pad1.20x1.40mm_HandSolder, F.Cu at (112.5, 99.8)
- added R52: 22.1k, Resistor_SMD:R_0805_2012Metric_Pad1.20x1.40mm_HandSolder, F.Cu at (81.8, 38.0)
- added R53: 47.5k, Resistor_SMD:R_0805_2012Metric_Pad1.20x1.40mm_HandSolder, F.Cu at (81.8, 42.0)
- added R54: 10K, Resistor_SMD:R_0805_2012Metric_Pad1.20x1.40mm_HandSolder, F.Cu at (55.5, 101.0)
- added R55: 10k, Resistor_SMD:R_0805_2012Metric_Pad1.20x1.40mm_HandSolder, F.Cu at (85.5, 37.0)
- added R56: 0.3k, Resistor_SMD:R_0805_2012Metric_Pad1.20x1.40mm_HandSolder, F.Cu at (85.5, 40.0)
- added R57: 0.3k, Resistor_SMD:R_0805_2012Metric_Pad1.20x1.40mm_HandSolder, F.Cu at (85.5, 43.0)
- added SW3: SW_Push_DPDT, dpdt_tht:dpdt, F.Cu at (151.0, 121.5)
- added SW4: SW_Push_DPDT, dpdt_tht:dpdt, F.Cu at (150.7, 91.8)
- added SW5: SW_Push_DPDT, dpdt_tht:dpdt, F.Cu at (150.8, 101.3)
- added SW6: SW_Push_DPDT, dpdt_tht:dpdt, F.Cu at (150.8, 111.5)
- added TP10: TP, TestPoint:TestPoint_Pad_D2.0mm, F.Cu at (168.4, 51.0)
- added TP11: TP, TestPoint:TestPoint_Pad_D2.0mm, F.Cu at (168.4, 55.0)
- added TP12: TP, TestPoint:TestPoint_Pad_D2.0mm, F.Cu at (168.4, 59.1)
- added TP13: TP, TestPoint:TestPoint_Pad_D2.0mm, F.Cu at (148.0, 28.2)
- added TP9: TP, TestPoint:TestPoint_Pad_D2.0mm, F.Cu at (164.3, 59.1)
- added U13: CP2102N-Axx-xQFN28, Package_DFN_QFN:QFN-28-1EP_5x5mm_P0.5mm_EP3.35x3.35mm, F.Cu at (75.5, 40.5)
- added U14: ESP32-WROOM-32U, RF_Module:ESP32-WROOM-32U, F.Cu at (62.9, 90.0)
- C10: value 100nF -> 0.1uF; footprint Capacitor_SMD:C_0805_2012Metric -> Capacitor_SMD:C_0805_2012Metric_Pad1.18x1.45mm_HandSolder
- C11, C12: value 100nF -> 0.1uF; footprint Capacitor_SMD:C_01005_0402Metric -> Capacitor_SMD:C_0805_2012Metric_Pad1.18x1.45mm_HandSolder
- C13, C14, C15, C16, C17, C2, C3, C4, C6, C8, C9: footprint Capacitor_SMD:C_0805_2012Metric -> Capacitor_SMD:C_0805_2012Metric_Pad1.18x1.45mm_HandSolder
- C18, C19, C22, C23, C24, C27: value 100n -> 0.1uF; footprint Capacitor_SMD:CP_Elec_6.3x7.7 -> Capacitor_SMD:C_0805_2012Metric_Pad1.18x1.45mm_HandSolder
- C20, C21, C25, C26: value 470u -> 470uF; footprint Capacitor_SMD:CP_Elec_6.3x7.7 -> Capacitor_SMD:CP_Elec_10x10.5
- C28: value 100n -> 10uF; footprint Capacitor_SMD:CP_Elec_6.3x7.7 -> Capacitor_SMD:C_0805_2012Metric_Pad1.18x1.45mm_HandSolder
- D10, D11, D13, D14, D15, D16, D17, D6, D7, D8: footprint LED_SMD:LED_0201_0603Metric_Pad0.64x0.40mm_HandSolder -> LED_SMD:LED_0805_2012Metric_Pad1.15x1.40mm_HandSolder
- J10, J5, J6, J7: footprint 2 Pin JST_Power&Motors:JST_B2B-XH-A_LF__SN_ -> Connector_JST:JST_EH_B2B-EH-A_1x02_P2.50mm_Vertical
- J2: footprint Connector_BarrelJack:BarrelJack_Wuerth_6941xx301002 -> Connector_BarrelJack:BarrelJack_GCT_DCJ200-10-A_Horizontal
- R1: value 10K -> 2k; footprint Resistor_SMD:R_0805_2012Metric -> Resistor_SMD:R_0805_2012Metric_Pad1.20x1.40mm_HandSolder
- R19, R20, R21, R22, R27, R30, R31, R32, R35, R40, R41, R42, R8, R9: footprint Resistor_SMD:R_0805_2012Metric -> Resistor_SMD:R_0805_2012Metric_Pad1.20x1.40mm_HandSolder
- R23, R24, R25, R26, R33, R34, R36, R37, R38, R39: footprint Resistor_SMD:R_0603_1608Metric -> Resistor_SMD:R_0805_2012Metric_Pad1.20x1.40mm_HandSolder
- R43, R44, R45, R46, R47, R48: value 100k -> 10k
- R6: footprint Resistor_SMD:R_0815_2038Metric -> Resistor_SMD:R_0805_2012Metric_Pad1.20x1.40mm_HandSolder
- moved D12 199.6 mm to (65.2, 33.8), turned to 90 degrees
- moved R28 198.9 mm to (61.2, 29.2)
- moved J10 197.0 mm to (239.0, 68.0), turned to -90 degrees
- moved R29 196.2 mm to (61.5, 42.2)
- moved R34 185.2 mm to (227.5, 69.2)
- moved Q1 182.3 mm to (180.8, 62.4), turned to 90 degrees
- moved R33 180.3 mm to (223.5, 69.2)
- moved D10 179.7 mm to (77.8, 70.0)
- moved D9 176.1 mm to (65.2, 39.5)
- moved J11 174.9 mm to (58.6, 35.9), turned to -90 degrees
- moved R30 172.6 mm to (77.8, 66.8), turned to 180 degrees
- moved U7 169.1 mm to (219.5, 57.8), turned to -90 degrees
- moved J12 168.5 mm to (238.8, 102.0), turned to 90 degrees
- moved J2 165.1 mm to (231.2, 40.6)
- moved H8 157.6 mm to (239.8, 26.2)
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Connections:
- J16 pad 1: /EB5 -> /EB1
- J16 pad 2: /EB4 -> /33
- J16 pad 3: /EB3 -> /32
- J17 pad 1: /EB2 -> /EB0
- J17 pad 2: /EB1 -> /35
- J17 pad 3: /EB0 -> /34
- J9 pad 3: unconnected-(J9-Pin_3-Pad3) -> /SHD
- J9 pad 4: unconnected-(J9-Pin_4-Pad4) -> /SWP
- J9 pad 5: unconnected-(J9-Pin_5-Pad5) -> /SCS
- J9 pad 6: unconnected-(J9-Pin_6-Pad6) -> /SCK
- J9 pad 7: unconnected-(J9-Pin_7-Pad7) -> /SD0
- J9 pad 8: unconnected-(J9-Pin_8-Pad8) -> /SD1
- R1 pad 1: /EN -> /3V3
- R1 pad 2: /3V3 -> Net-(U13-~{RST})
- R16 pad 2: /3.3V -> /3V3
- R17 pad 2: /3.3V -> /3V3
- R18 pad 2: /3.3V -> /3V3
- R44 pad 1: Net-(U12-INTA) -> /3V3
- R44 pad 2: /3V3 -> Net-(U12-INTA)
- R45 pad 2: /3V3 -> Net-(JP1-A)
- R46 pad 2: /3V3 -> Net-(JP2-A)
- R47 pad 2: /3V3 -> Net-(JP3-A)
- R48 pad 1: Net-(U12-~{RESET}) -> /3V3
- R48 pad 2: /3V3 -> Net-(U12-~{RESET})
- TH1 pad 1: Net-(J3-Pin_3) -> /12V_P
- U10 pad 2: /EA0 -> /26
- U10 pad 3: /EA1 -> /EA0
- U10 pad 4: /EA2 -> /27
- U10 pad 5: /EA3 -> /EA1
- U10 pad 6: /EA4 -> /25
- U10 pad 7: /EA5 -> /EA2
- U11 pad 2: /23 -> /EB2
- U11 pad 3: /25 -> /EB3
- U11 pad 4: /26 -> /EB4
- U12 pad 12: /22 -> /SD1
- U12 pad 13: /21 -> /SD0
- U12 pad 15: /3V3 -> Net-(JP1-A)
- U12 pad 16: /3V3 -> Net-(JP2-A)
- U12 pad 17: /3V3 -> Net-(JP3-A)
- U5 pad 10: unconnected-(U5-~{FLT}-Pad10) -> /FLT/VIO3
- U5 pad 4: /3V3 -> /M2/NC
- U5 pad 5: /3V3 -> /RST/PDN
- U5 pad 6: /3V3 -> /SLP/CLK
- U6 pad 10: unconnected-(U6-~{FLT}-Pad10) -> /FLT/VIO1
- U6 pad 4: /3V3 -> /M2/NC
- U6 pad 5: /3V3 -> /RST/PDN
- U6 pad 6: /3V3 -> /SLP/CLK
- U8 pad 10: unconnected-(U8-~{FLT}-Pad10) -> /FLT/VIO2
- U8 pad 4: /3V3 -> /M2/NC
- U8 pad 5: /3V3 -> /RST/PDN
- U8 pad 6: /3V3 -> /SLP/CLK
- U9 pad 10: unconnected-(U9-~{FLT}-Pad10) -> /FLT/VIO4
- U9 pad 4: /3V3 -> /M2/NC
- U9 pad 5: /3V3 -> /RST/PDN
- U9 pad 6: /3V3 -> /SLP/CLK
Routing:
- net /3V3: track 346.9 -> 0.00 mm, vias 3 -> 0
- net /12V_P: track 231.0 -> 0.00 mm
- net /5V: track 197.9 -> 0.00 mm
- net (no net): track 134.1 -> 0.00 mm
- net /EN: track 132.2 -> 0.00 mm, vias 2 -> 0
- net /25: track 127.3 -> 0.00 mm
- net /26: track 124.2 -> 0.00 mm
- net /35: track 109.4 -> 0.00 mm, vias 1 -> 0
- net /34: track 103.4 -> 0.00 mm, vias 1 -> 0
- net /4: track 99.7 -> 0.00 mm, vias 1 -> 0
- net /15: track 99.0 -> 0.00 mm
- net /14: track 96.8 -> 0.00 mm
- net /22: track 94.8 -> 0.00 mm
- net /18: track 93.3 -> 0.00 mm
- net /23: track 92.6 -> 0.00 mm
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- removed copper zone on B.Cu, net GND
- removed copper zone on F.Cu, net GND
Other:
- board size 120 x 120 mm -> 190.5 x 121.8 mm
